File: Platine/KNX_BOH.kicad_pcb (KiCad board)
At the start: 2 copper layers, 25 parts, among them K1 FINDER-40.41, K2 FINDER-40.41, K3 FINDER-40.41, K4 FINDER-40.41, K5 FINDER-40.41, K6 FINDER-40.41, K7 FINDER-40.41, Q1 BC547, Q2 BC547, Q3 BC547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

Commit message: Platine fast fertig
Parts:
- removed the D1 at (52.4, 8.52)
- removed the D1 at (72.8, 81.5)
- removed D7: D, Diode_THT:D_A-405_P10.16mm_Horizontal
- removed the K1 at (91.5, 84.5)
- removed the K1 at (54.7, -4.28)
- removed K7: FINDER-40.41, Relay_THT:Relay_SPDT_Finder_40.41
- removed the Q1 at (66.2, 9.65)
- removed the Q1 at (89.5, 98.4)
- removed Q7: BC547, Package_TO_SOT_THT:TO-92_Inline
- added ChipReader1: Screw_Terminal_01x07, TerminalBlock_Phoenix:TerminalBlock_Phoenix_MKDS-1,5-7-5.08_1x07_P5.08mm_Horizontal, F.Cu at (140.0, 82.5)
- added D1: D, Diode_THT:D_A-405_P10.16mm_Horizontal, F.Cu at (177.7, 56.6)
- added DotMatrixDoor1: Screw_Terminal_01x05, TerminalBlock_Phoenix:TerminalBlock_Phoenix_MPT-0,5-7-2.54_1x07_P2.54mm_Horizontal, F.Cu at (118.7, 80.4)
- added DotMatrixGarage1: Screw_Terminal_01x05, TerminalBlock_Phoenix:TerminalBlock_Phoenix_MPT-0,5-7-2.54_1x07_P2.54mm_Horizontal, F.Cu at (118.7, 88.7)
- added DotMatrixRollo1: Screw_Terminal_01x05, TerminalBlock_Phoenix:TerminalBlock_Phoenix_MPT-0,5-7-2.54_1x07_P2.54mm_Horizontal, F.Cu at (118.7, 96.9)
- added DotMatrixRollo2: Screw_Terminal_01x05, TerminalBlock_Phoenix:TerminalBlock_Phoenix_MPT-0,5-7-2.54_1x07_P2.54mm_Horizontal, F.Cu at (118.7, 105.2)
- added DotMatrixWindow1: Screw_Terminal_01x05, TerminalBlock_Phoenix:TerminalBlock_Phoenix_MPT-0,5-7-2.54_1x07_P2.54mm_Horizontal, F.Cu at (118.7, 113.4)
- added Garage1: Screw_Terminal_01x02, TerminalBlock_Phoenix:TerminalBlock_Phoenix_MKDS-1,5-2-5.08_1x02_P5.08mm_Horizontal, F.Cu at (119.7, 46.9)
- added Garage2: Screw_Terminal_01x02, TerminalBlock_Phoenix:TerminalBlock_Phoenix_MKDS-1,5-2-5.08_1x02_P5.08mm_Horizontal, F.Cu at (119.7, 58.8)
- added Interaktion1: Screw_Terminal_01x02, TerminalBlock_Phoenix:TerminalBlock_Phoenix_MKDS-1,5-2-5.08_1x02_P5.08mm_Horizontal, F.Cu at (119.7, 70.7)
- added J1: Conn_01x04_Pin, TerminalBlock_Phoenix:TerminalBlock_Phoenix_MKDS-3-4-5.08_1x04_P5.08mm_Horizontal, F.Cu at (225.6, 113.0)
- added J2: Conn_01x04_Pin, TerminalBlock_Phoenix:TerminalBlock_Phoenix_MKDS-3-4-5.08_1x04_P5.08mm_Horizontal, F.Cu at (203.1, 113.0)
- added K1: DSBT2-S-DC24V, BOH_KNX:DSBT2SDC24V, F.Cu at (140.6, 130.3)
- added KNXDoor1: Screw_Terminal_01x02, TerminalBlock_Phoenix:TerminalBlock_Phoenix_MKDS-1,5-2-5.08_1x02_P5.08mm_Horizontal, F.Cu at (131.9, 46.9)
- added KNXDoorChip1: Screw_Terminal_01x02, TerminalBlock_Phoenix:TerminalBlock_Phoenix_MKDS-1,5-2-5.08_1x02_P5.08mm_Horizontal, F.Cu at (131.9, 58.8)
- added KNXGarage1: Screw_Terminal_01x02, TerminalBlock_Phoenix:TerminalBlock_Phoenix_MKDS-1,5-2-5.08_1x02_P5.08mm_Horizontal, F.Cu at (131.9, 70.7)
- added KNXRaining1: Screw_Terminal_01x02, TerminalBlock_Phoenix:TerminalBlock_Phoenix_MKDS-1,5-2-5.08_1x02_P5.08mm_Horizontal, F.Cu at (144.1, 46.9)
- added KNXWind1: Screw_Terminal_01x02, TerminalBlock_Phoenix:TerminalBlock_Phoenix_MKDS-1,5-2-5.08_1x02_P5.08mm_Horizontal, F.Cu at (144.1, 58.8)
- added KNXWindow1: Screw_Terminal_01x02, TerminalBlock_Phoenix:TerminalBlock_Phoenix_MKDS-1,5-2-5.08_1x02_P5.08mm_Horizontal, F.Cu at (144.1, 70.7)
- added KNX_COM1: Screw_Terminal_01x02, TerminalBlock_Phoenix:TerminalBlock_Phoenix_MKDS-1,5-2-5.08_1x02_P5.08mm_Horizontal, F.Cu at (156.4, 46.9)
- added LedStripe1: Screw_Terminal_01x03, TerminalBlock_Phoenix:TerminalBlock_Phoenix_MKDS-1,5-3-5.08_1x03_P5.08mm_Horizontal, F.Cu at (140.0, 94.4)
- added Q1: BC547, Package_TO_SOT_THT:TO-92_Inline, F.Cu at (191.6, 57.7)
- added ROLLO1: Screw_Terminal_01x02, TerminalBlock_Phoenix:TerminalBlock_Phoenix_MKDS-1,5-2-5.08_1x02_P5.08mm_Horizontal, F.Cu at (156.4, 58.8)
- added ROLLO2: Screw_Terminal_01x02, TerminalBlock_Phoenix:TerminalBlock_Phoenix_MKDS-1,5-2-5.08_1x02_P5.08mm_Horizontal, F.Cu at (156.4, 70.7)
- K2, K3, K4, K5, K6: value FINDER-40.41 -> DSBT2-S-DC24V; footprint Relay_THT:Relay_SPDT_Finder_40.41 -> BOH_KNX:DSBT2SDC24V
- moved K3 136.2 mm to (179.0, 94.6)
- moved D2 129.9 mm to (177.7, 99.7)
- moved Q2 129.9 mm to (191.6, 100.8)
- moved K6 116.2 mm to (114.9, 130.3)
- moved D6 109.0 mm to (113.5, 135.4)
- moved Q6 109.0 mm to (127.4, 136.5)
- moved K2 107.2 mm to (179.0, 51.5)
- moved D4 96.2 mm to (177.7, 78.1)
- moved Q4 96.2 mm to (191.6, 79.3)
- moved K4 91.3 mm to (89.1, 130.3)
- moved D3 90.8 mm to (87.8, 135.4)
- moved Q3 90.8 mm to (101.6, 136.5)
- moved D5 89.6 mm to (139.3, 135.4)
- moved K5 88.2 mm to (179.0, 73.0)
- moved Q5 87.5 mm to (153.1, 136.5)
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Connections:
- net Regen_KNX renamed KNXRain
- net Rollo_1_KNX renamed KNXDoor
- net Rollo_2_KNX renamed KNXDoorChip
- net Rollo_3_KNX renamed KNXGarage
- net Rollo_4_KNX renamed KNXWindow
- K2 pad 11: KNX_COM -> Net-(K2-N.C._1)
- K3 pad 11: KNX_COM -> Net-(K3-N.C._1)
- K4 pad 11: KNX_COM -> Net-(K4-N.C._1)
- K5 pad 11: KNX_COM -> Net-(K5-N.C._1)
- K6 pad 11: KNX_COM -> Net-(K6-N.C._1)
- U2 pad J2-1: unconnected-(U2-3V3-PadJ2-1) -> +3V3
- U2 pad J2-19: unconnected-(U2-EXT_5V-PadJ2-19) -> +5V
- U2 pad J2-5: unconnected-(U2-IO34-PadJ2-5) -> Rain_Automatic
- U2 pad J2-6: unconnected-(U2-IO35-PadJ2-6) -> Rain_Manual
- U2 pad J2-7: unconnected-(U2-IO32-PadJ2-7) -> Wind_Automatic
- U2 pad J2-8: unconnected-(U2-IO33-PadJ2-8) -> Wind_Manual
- U2 pad J3-10: unconnected-(U2-IO5-PadJ3-10) -> CC
- U2 pad J3-2: unconnected-(U2-IO23-PadJ3-2) -> MOSI
- U2 pad J3-8: unconnected-(U2-IO19-PadJ3-8) -> MISO
- U2 pad J3-9: unconnected-(U2-IO18-PadJ3-9) -> SCK

Commit message: finished schematic
Parts:
- removed Garage2: Screw_Terminal_01x02, TerminalBlock_Phoenix:TerminalBlock_Phoenix_MKDS-1,5-2-5.08_1x02_P5.08mm_Horizontal
- removed U2: ESP32-DEVKITC-32D, ESP32-DEVKITC-32D:esp32_dev
- added Door1: Screw_Terminal_01x02, TerminalBlock_Phoenix:TerminalBlock_Phoenix_MKDS-1,5-2-5.08_1x02_P5.08mm_Horizontal, F.Cu at (150.5, 46.7)
- added ESP32_WROOM_32D_USB-C2: ~, bulme_footprints:ESP32_WROOM_32D_USB-C, F.Cu at (60.0, 72.5)
- added R1: 10k, Resistor_THT:R_Axial_DIN0207_L6.3mm_D2.5mm_P10.16mm_Horizontal, F.Cu at (168.8, 101.8)
- added R2: 10k, Resistor_THT:R_Axial_DIN0207_L6.3mm_D2.5mm_P10.16mm_Horizontal, F.Cu at (168.8, 105.9)
- added R3: 10k, Resistor_THT:R_Axial_DIN0207_L6.3mm_D2.5mm_P10.16mm_Horizontal, F.Cu at (168.8, 109.9)
- added R4: 10k, Resistor_THT:R_Axial_DIN0207_L6.3mm_D2.5mm_P10.16mm_Horizontal, F.Cu at (168.8, 114.0)
- K1, K2, K3, K4, K5, K6: footprint BOH_KNX:DSBT2SDC24V -> bulme_footprints:DSBT2SDC24V
- moved Garage1 32.9 mm to (150.5, 58.6)
- moved D5 30.8 mm to (170.1, 135.2)
- moved K1 30.8 mm to (171.4, 130.1)
- moved K2 30.8 mm to (209.8, 51.3)
- moved K3 30.8 mm to (209.8, 94.4)
- moved K5 30.8 mm to (209.8, 72.8)
- moved D6 30.8 mm to (144.3, 135.2)
- moved Interaktion1 30.8 mm to (150.5, 70.5)
- moved K6 30.8 mm to (145.6, 130.1)
- moved Q3 30.8 mm to (132.4, 136.3)
- moved Q6 30.8 mm to (158.1, 136.3)
- moved ChipReader1 30.8 mm to (170.8, 82.3)
- moved D1 30.8 mm to (208.5, 56.4)
- moved D2 30.8 mm to (208.5, 99.5)
- moved D3 30.8 mm to (118.5, 135.2)
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Connections:
- Garage1 pad 1: KNX_Garage -> KNX_Garage_UP
- Garage1 pad 2: KNX_Garage -> KNX_Garage_DOWN
