File: Platine/Relais.kicad_sch (KiCad schematic)
At the start: 3 parts, among them K5 FINDER-40.41, Q5 BC547

Commit message: Platine fast fertig
Parts:
- removed K5: FINDER-40.41, Relay_THT:Relay_SPDT_Finder_40.41, symbol Relay:FINDER-40.41
- added K4: DSBT2-S-DC24V, DSBT2SDC24V, symbol BOH_KNX:DSBT2-S-DC24V
Connections:
- net GND: now also K4.16 (COIL-)
- net Relais_COM: now also K4.13 (COM_2), K4.4 (COM_1)
- net Relais_OUT: now also K4.8 (N.O._1), K4.9 (N.O._2)
- net at D5.1 (K), Q5.3 (E): now also K4.1 (COIL+)
- new net: K4.11 (N.C._2), K4.6 (N.C._1)
Other:
- moved on the sheet: Q5

Commit message: finished schematic
Parts:
- K4: footprint DSBT2SDC24V -> bulme_footprints:DSBT2SDC24V
- renumbered D5 to D3, Q5 to Q3
Changed lines of the file:
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@@
 		(dnp no)
 		(fields_autoplaced yes)
-		(property "Reference" "#PWR011"
+		(property "Reference" "#PWR07"
 			(at 139.7 74.93 0)
 			(effects
@@
 		(dnp no)
 		(fields_autoplaced yes)
-		(property "Reference" "D5"
+		(property "Reference" "D3"
 			(at 142.24 92.7099 90)
 			(effects
@@
 		(dnp no)
 		(fields_autoplaced yes)
-		(property "Reference" "Q5"
+		(property "Reference" "Q3"
 			(at 142.24 78.7399 0)
 			(effects
@@
 			)
 		)
-		(property "Footprint" "DSBT2SDC24V"
+		(property "Footprint" "bulme_footprints:DSBT2SDC24V"
 			(at 179.07 187.63 0)
 			(effects
@@
 		(dnp no)
 		(fields_autoplaced yes)
-		(property "Reference" "#PWR015"
+		(property "Reference" "#PWR08"
 			(at 139.7 111.76 0)
 			(effects
