File: Platine/select.kicad_sch (KiCad schematic)
At the start: 3 parts

Commit message: Platine fast fertig
Parts:
- removed R2: 10kR, Resistor_SMD:R_1206_3216Metric, symbol Device:R
- removed Sel_Auto, Sel_ON/OFF: SW_Nidec_CAS-120A1, symbol Switch:SW_Nidec_CAS-120A1
- added J2: Conn_01x04_Pin, TerminalBlock_Phoenix:TerminalBlock_Phoenix_MKDS-3-4-5.08_1x04_P5.08mm_Horizontal, symbol Connector:Conn_01x04_Pin
Connections:
- net Automatic: now also J2.1 (Pin_1)
- net GND: now also J2.4 (Pin_4)
- net Manuell_OFF: now also J2.2 (Pin_2)
- net Manuell_ON: now also J2.3 (Pin_3)

Commit message: finished schematic
Parts:
- renumbered J2 to J1
Changed lines of the file:
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@@
 		(dnp no)
 		(fields_autoplaced yes)
-		(property "Reference" "J2"
+		(property "Reference" "J1"
 			(at 144.78 90.17 90)
 			(effects
